Commit message: updated urdf transdforms

File: rr_description/urdf/evgp.urdf.xacro (robot description, xacro)
@@ -97,5 +97,5 @@
     </link>
     <xacro:set_link_color link="camera" color="Gold"/>
-    <link name="imu_link">
+    <link name="imu_top_link">
         <xacro:null_inertia/>
         <visual>
@@ -105,5 +105,5 @@
         </visual>
     </link>
-    <xacro:set_link_color link="imu_link" color="Gold"/>
+    <xacro:set_link_color link="imu_top_link" color="Gold"/>
     <!-- ************************** Joints *************************** -->
     <xacro:property name="joint_flop_both" value="0.03"/>
@@ -143,15 +143,15 @@
         <parent link="base_footprint"/>
         <child link="lidar"/>
-        <origin xyz="1.2 0 0.18" rpy="0 0 0"/>
+        <origin xyz="1.1684 0 0.2286" rpy="0 0 0"/>
     </joint>
     <joint name="base_footprint_to_gps" type="fixed">
         <parent link="base_footprint"/>
         <child link="gps_link"/>
-        <origin xyz="0.5 0.5 0.1" rpy="0 0 0"/>
+        <origin xyz="0.4318 0.5588 1.27" rpy="0 0 0"/>
     </joint>
     <joint name="base_footprint_to_camera" type="fixed">
         <parent link="base_footprint"/>
         <child link="camera"/>
-        <origin xyz="0.1 0 0.7" rpy="0 0.2 0"/>
+        <origin xyz="0.4318 0.5588 1.0922" rpy="0 0.2 0"/>
     </joint>
     <xacro:macro name="camera_optical_frame" params="camera_link">
@@ -166,8 +166,8 @@
     </xacro:macro>
     <xacro:camera_optical_frame camera_link="camera"/>
-    <joint name="base_footprint_to_imu" type="fixed">
+    <joint name="base_footprint_to_imu_top" type="fixed">
         <parent link="base_footprint"/>
-        <child link="imu_link"/>
-        <origin xyz="0.75 0.5 0.1" rpy="0 0 0"/>
+        <child link="imu_top_link"/>
+        <origin xyz="0.4318 0.5588 0.9906" rpy="0 0 0"/>
     </joint>
     <!-- ******************* Sensors *********************** -->
@@ -242,7 +242,7 @@
 <!--    </gazebo>-->
     <!-- IMU -->
-    <gazebo reference="imu_link">
+    <gazebo reference="imu_top_link">
         <gravity>true</gravity>
-        <sensor name="imu_sensor" type="imu">
+        <sensor name="imu_top_sensor" type="imu">
             <always_on>true</always_on>
             <update_rate>100</update_rate>
@@ -250,11 +250,11 @@
             <topic>__default_topic__</topic>
             <plugin filename="libgazebo_ros_imu_sensor.so" name="imu_plugin">
-                <topicName>imu</topicName>
-                <bodyName>imu_link</bodyName>
+                <topicName>imu_top</topicName>
+                <bodyName>imu_top_link</bodyName>
                 <updateRateHZ>20.0</updateRateHZ>
                 <gaussianNoise>0.005</gaussianNoise>
                 <xyzOffset>0 0 0</xyzOffset>
                 <rpyOffset>0 0 0</rpyOffset>
-                <frameName>imu_link</frameName>
+                <frameName>imu_top_link</frameName>
             </plugin>
             <pose>0 0 0 0 0 0</pose>

Commit message: testing localization, imu rotation messed up

File: rr_description/urdf/evgp.urdf.xacro (robot description, xacro)
@@ -97,5 +97,5 @@
     </link>
     <xacro:set_link_color link="camera" color="Gold"/>
-    <link name="imu_top_link">
+    <link name="imu_top">
         <xacro:null_inertia/>
         <visual>
@@ -105,5 +105,5 @@
         </visual>
     </link>
-    <xacro:set_link_color link="imu_top_link" color="Gold"/>
+    <xacro:set_link_color link="imu_top" color="Gold"/>
     <!-- ************************** Joints *************************** -->
     <xacro:property name="joint_flop_both" value="0.03"/>
@@ -168,6 +168,6 @@
     <joint name="base_footprint_to_imu_top" type="fixed">
         <parent link="base_footprint"/>
-        <child link="imu_top_link"/>
-        <origin xyz="0.4318 0.5588 0.9906" rpy="0 0 0"/>
+        <child link="imu_top"/>
+        <origin xyz="0.4318 0.5588 0.9906" rpy="${pi/2} 0 0"/>
     </joint>
     <!-- ******************* Sensors *********************** -->
